Commit message: Fix URDF

File: jaka_kargo_ros2/src/jaka_kargo_description/urdf/jaka_kargo.urdf (robot description, URDF)
Before this commit: robot jaka_kargo, 31 links, 30 joints
Links:
- link body_j1_link: mass 0 -> 12.252

Commit message: Update URDF

File: jaka_kargo_ros2/src/jaka_kargo_description/urdf/jaka_kargo.urdf (robot description, URDF)
Before this commit: robot jaka_kargo, 31 links, 30 joints
Links:
- link arm_lj1_link: mass 0.55668 -> 0.556662347813903
- link arm_lj2_link: mass 0.96177 -> 0.961807814148841
- link arm_lj4_link: mass 0.52447 -> 0.524473557771922
- link arm_lj5_link: mass 0.79519 -> 0.79516120070511
- link arm_lj6_link: mass 0.57658 -> 0.576577893328044
- link arm_lj7_link: mass 0.23674 -> 0.236737677400848
- link arm_rj1_link: mass 0.55667 -> 0.55666
- link arm_rj2_link: mass 0.96177 -> 0.96181
- link arm_rj5_link: mass 0.79519 -> 0.79516
- link body_j1_link: mass 12.252 -> 14.555
- link body_j2_link: mass 5.4288 -> 11.807
- link body_j3_link: mass 0.81199 -> 2.1924
- link camera_1_link: mass 0.087598 -> 0.089349902292875
- link camera_2_link: mass 0.087598 -> 0.0893499022928749
- link h_wheel_q_link: mass 0.79441 -> 0.794411429544822
- link h_wheel_w_link: mass 0.39912 -> 0.399115828829937
- link h_wheel_x_link: mass 2.1992 -> 0.785339554840708
- link q_wheel_w_link: mass 0.39912 -> 0.399115828829937
- link q_wheel_x_link: mass 2.1992 -> 0.785339554840708
- link radar_3d_link: mass 0.0093217 -> 0.00950816080674812
- link radar_l_link: mass 0.017051 -> 0.0173915767921935
- link radar_r_link: mass 0.017051 -> 0.0173915767921936
Joints:
- joint arm_lj2: origin xyz=0 0 0.203 rpy=-1.5708 0 -1.5708 -> xyz=0 0 0.203 rpy=-1.5708 0 0
- joint arm_lj3: origin xyz=0 0 0 rpy=1.5708 0 -1.5708 -> xyz=0 0 0 rpy=1.5708 0 0
- joint arm_lj4: limit lower=-2.53073 upper=0.5236 effort=0 velocity=2.0944 -> lower=-2.531 upper=0.5236 effort=0 velocity=2.0944; origin xyz=0.00040027 -0.00039997 -0.3415 rpy=1.5708 0 0 -> xyz=-0.00040027 0.0004006 0.3415 rpy=-1.5708 0 0
- joint arm_rj1: origin xyz=-0.0047083 0.24 -0.0497 rpy=-3.1416 -0.5236 -3.1416  -> xyz=-0.0047083 0.24 -0.0497 rpy=3.1416 -0.5236 -3.1416
- joint arm_rj2: origin xyz=0 0 0.203 rpy=-1.5708 0 -1.5708  -> xyz=0 0 0.203 rpy=-1.5708 0 -3.1416
- joint arm_rj3: origin xyz=0 0 0 rpy=1.5708 -1.0472 -1.5708 -> xyz=0 0 0 rpy=1.5708 0 0
- joint arm_rj4: limit lower=-2.53073 upper=0.5236 effort=0 velocity=2.0944 -> lower=-2.531 upper=0.5236 effort=0 velocity=2.0944; origin xyz=-0.00014624 -0.00054663 -0.3415 rpy=1.5708 0 -1.0472 -> xyz=-0.00040027 0.0004006 0.3415 rpy=-1.5708 0 0
- joint arm_rj6: origin xyz=0 -0.00039946 0.23194 rpy=-1.5708 0 0 -> xyz=0 -0.00040035 0.23194 rpy=-1.5708 0 -3.1416
- joint body_j4: axis 0 0 1 -> 0 0 -1; limit lower=0 upper=0.6981 effort=0 velocity=0 -> lower=-0.3491 upper=0.7854 effort=0 velocity=0; origin xyz=1.6525E-05 0.0002 0.095 rpy=1.5708 0 3.0592 -> xyz=1.6524729565065E-05 0.000200000000069326 0.0949999999999905 rpy=1.5707963267949 0 3.05915625416187
- joint wheel_1: axis 0 0 1 -> 0 0 -1
- joint wheel_2: origin xyz=-0.29 -0.1975 0.006 rpy=1.5708 0 -3.1416 -> xyz=-0.29 -0.175 0.006 rpy=1.5708 -0.44445 3.1416
- joint wheel_3: axis 0 0 1 -> 0 0 -1; origin xyz=0.29 0.1975 0.145 rpy=0 0 0 -> xyz=0.29 0.1975 0.145 rpy=3.1416 0 3.1416
- joint wheel_4: axis 0 0 1 -> 0 0 -1; origin xyz=-0.29 -0.1975 0.145 rpy=0 0 0 -> xyz=-0.29 -0.1975 0.145 rpy=3.1416 0 0

Commit message: AGV MoveIt implementation

File: jaka_kargo_ros2/src/jaka_kargo_description/urdf/jaka_kargo.urdf (robot description, URDF)
Before this commit: robot jaka_kargo, 31 links, 30 joints
Links:
- added link agv_x_link
- added link agv_xy_link
- added link arm_l_tcp
- added link arm_r_tcp
- link arm_lj1_link: mass 0.556662347813903 -> 0.556662347813916
- link arm_lj2_link: mass 0.961807814148841 -> 0.961807814148781
- link arm_lj3_link: mass 1.3625 -> 1.3625354645121
- link arm_lj4_link: mass 0.524473557771922 -> 0.524473517277118
- link arm_lj5_link: mass 0.79516120070511 -> 0.795161200903781
- link arm_lj6_link: mass 0.576577893328044 -> 0.576577893328043
- link arm_rj1_link: mass 0.55666 -> 0.556662347813879
- link arm_rj2_link: mass 0.96181 -> 0.961807814148782
- link arm_rj3_link: mass 1.3625 -> 1.36253546451272
- link arm_rj4_link: mass 0.52447 -> 0.524473554546553
- link arm_rj5_link: mass 0.79516 -> 0.795157721674083
- link arm_rj6_link: mass 0.57658 -> 0.576576632917431
- link arm_rj7_link: mass 0.23674 -> 0.236737677400848
- link base_link: mass 130.51 -> 130.512640281208
- link body_j1_link: mass 14.555 -> 14.5550705585876
- link body_j2_link: mass 11.807 -> 11.8071087615657
- link body_j3_link: mass 2.1924 -> 2.1923611998553
- link body_j4_link: mass 0.62325 -> 0.623251763320113
- link q_wheel_q_link: mass 0.79441 -> 0.794411429544822
Joints:
- removed joint fixed
- added joint agv_x: type prismatic, parent world, child agv_x_link, origin xyz=0 0 0 rpy=0 0 0, axis 1 0 0, limit lower=-20.0 upper=20.0 effort=1000 velocity=0.5
- added joint agv_y: type prismatic, parent agv_x_link, child agv_xy_link, origin xyz=0 0 0 rpy=0 0 0, axis 0 1 0, limit lower=-20.0 upper=20.0 effort=1000 velocity=0.5
- added joint agv_yaw: type revolute, parent agv_xy_link, child base_link, origin xyz=0 0 0 rpy=0 0 0, axis 0 0 1, limit lower=-3.1415926 upper=3.1415926 effort=1000 velocity=1.57
- added joint arm_l_tcp_joint: type fixed, parent arm_lj7_link, child arm_l_tcp, origin xyz=0 0 0.2 rpy=0 0 0
- added joint arm_r_tcp_joint: type fixed, parent arm_rj7_link, child arm_r_tcp, origin xyz=0 0 0.2 rpy=0 0 0
- joint arm_lj1: limit lower=-6.2832 upper=6.2832 effort=0 velocity=1.5708 -> lower=-6.2832 upper=6.2832 effort=66 velocity=1.5708; origin xyz=-0.0047083 0.24 0.0493 rpy=0 -0.5236 0 -> xyz=0.00470834833564851 -0.239999999669298 0.0492999999991973 rpy=0 -0.523598775600649 3.14159265358979
- joint arm_lj2: limit lower=-1.8326 upper=1.8326 effort=0 velocity=1.5708 -> lower=-1.8326 upper=1.8326 effort=66 velocity=1.5708; origin xyz=0 0 0.203 rpy=-1.5708 0 0 -> xyz=0 0 0.202999999999558 rpy=-1.5707963267949 0 0
- joint arm_lj3: limit lower=-6.2832 upper=6.2832 effort=0 velocity=2.0944 -> lower=-6.2832 upper=6.2832 effort=64 velocity=2.0944; origin xyz=0 0 0 rpy=1.5708 0 0 -> xyz=0 0 0 rpy=1.57079746215332 0 0
- joint arm_lj4: limit lower=-2.531 upper=0.5236 effort=0 velocity=2.0944 -> lower=-2.3562 upper=0.5236 effort=37 velocity=2.0944; origin xyz=-0.00040027 0.0004006 0.3415 rpy=-1.5708 0 0 -> xyz=-0.000400273519917158 0.000400600664341555 0.341500117255216 rpy=-1.5707963267949 0 0
- joint arm_lj5: limit lower=-6.2832 upper=6.2832 effort=0 velocity=2.618 -> lower=-6.2832 upper=6.2832 effort=19 velocity=2.618; origin xyz=0 0 0 rpy=1.5708 0 0 -> xyz=0 0 0 rpy=1.57079662831086 0 0
- joint arm_lj6: limit lower=-1.8326 upper=1.8326 effort=0 velocity=2.618 -> lower=-1.8326 upper=1.8326 effort=19 velocity=2.618; origin xyz=0 -0.00039946 0.23194 rpy=-1.5708 0 0 -> xyz=0 -0.00213275470159946 0.231935198030176 rpy=-1.5707963267949 0 0
- joint arm_lj7: limit lower=-6.2832 upper=6.2832 effort=0 velocity=2.618 -> lower=-6.2832 upper=6.2832 effort=19 velocity=2.618; origin xyz=0 0 0 rpy=1.5708 0 0 -> xyz=0 0 0 rpy=1.5707963267949 0 0
- joint arm_rj1: limit lower=-6.2832 upper=6.2832 effort=0 velocity=1.5708 -> lower=-6.2832 upper=6.2832 effort=66 velocity=1.5708; origin xyz=-0.0047083 0.24 -0.0497 rpy=3.1416 -0.5236 -3.1416 -> xyz=0.00470834833541592 -0.239999999669298 -0.0497000000008027 rpy=3.14159265234577 -0.52359877559595 0
- joint arm_rj2: limit lower=-1.8326 upper=1.8326 effort=0 velocity=1.5708 -> lower=-1.8326 upper=1.8326 effort=66 velocity=1.5708; origin xyz=0 0 0.203 rpy=-1.5708 0 -3.1416 -> xyz=0 0 0.202999999999558 rpy=-1.5707963267949 0 -3.14159265305106
- joint arm_rj3: limit lower=-6.2832 upper=6.2832 effort=0 velocity=2.0944 -> lower=-6.2832 upper=6.2832 effort=64 velocity=2.0944; origin xyz=0 0 0 rpy=1.5708 0 0 -> xyz=0 0 0 rpy=1.57079746215332 0 0
- joint arm_rj4: limit lower=-2.531 upper=0.5236 effort=0 velocity=2.0944 -> lower=-2.3562 upper=0.5236 effort=37 velocity=2.0944; origin xyz=-0.00040027 0.0004006 0.3415 rpy=-1.5708 0 0 -> xyz=-0.000400273782725766 0.000400599423920567 0.341500117255216 rpy=-1.5707963267949 0 0
- joint arm_rj5: limit lower=-6.2832 upper=6.2832 effort=0 velocity=2.618 -> lower=-6.2832 upper=6.2832 effort=19 velocity=2.618; origin xyz=0 0 0 rpy=1.5708 0 0 -> xyz=0 0 0 rpy=1.57079662831086 0 0
- joint arm_rj6: limit lower=-1.8326 upper=1.8326 effort=0 velocity=2.618 -> lower=-1.8326 upper=1.8326 effort=19 velocity=2.618; origin xyz=0 -0.00040035 0.23194 rpy=-1.5708 0 -3.1416 -> xyz=0 0.00133294267563855 0.231935198030161 rpy=-1.5707963267949 0 -3.14159249457812
- joint arm_rj7: limit lower=-6.2832 upper=6.2832 effort=0 velocity=2.618 -> lower=-6.2832 upper=6.2832 effort=19 velocity=2.618; origin xyz=0 0 0 rpy=1.5708 0 0 -> xyz=0 0 0 rpy=1.5707963267949 0 0
- joint body_j1: axis 0 0 1 -> 1 0 0; limit lower=0 upper=0.8 effort=0 velocity=0 -> lower=0 upper=0.78 effort=1350 velocity=0.1; origin xyz=0.005341 0 0.309 rpy=0 0 0 -> xyz=0.018341 0 0.1943 rpy=-3.1416 -1.5708 0
- joint body_j2: limit lower=0 upper=1.5707 effort=0 velocity=0 -> lower=0 upper=1.5707 effort=281 velocity=1.5708; origin xyz=0.15 0 0.1175 rpy=1.5708 0 3.1416 -> xyz=0 0 0 rpy=1.5708 -1.5708 0
- joint body_j3: limit lower=-1.5707 upper=1.5707 effort=0 velocity=0 -> lower=-1.5707 upper=1.5707 effort=19 velocity=1.5708; origin xyz=0 0.3054 -0.0002 rpy=1.5708 0 3.1416 -> xyz=0 -0.3054 -0.0002 rpy=1.5708 0 0
- joint body_j4: limit lower=-0.3491 upper=0.7854 effort=0 velocity=0 -> lower=-0.3491 upper=0.7854 effort=19 velocity=1.5708; origin xyz=1.6524729565065E-05 0.000200000000069326 0.0949999999999905 rpy=1.5707963267949 0 3.05915625416187 -> xyz=1.65247295646487E-05 0.000200000000064386 0.0949999999999904 rpy=-1.5707963267949 0 -0.0824363994279264
- joint camera_1: origin xyz=-0.061 0.119 -0.0002 rpy=1.5708 0 -1.5708 -> xyz=0.061 -0.119 -0.0002 rpy=1.5708 0 1.5708
- joint camera_2: origin xyz=-0.034 0.053 -0.00020068 rpy=1.5708 0 -1.5708 -> xyz=0.0339999999999933 -0.0530000000000007 -0.000200681505657571 rpy=1.5707963267949 0 1.5707963267949
- joint radar_1: origin xyz=0.3262 -0.2262 0.217 rpy=0 0 0 -> xyz=0.18919999999982 -0.226200000000231 -0.0270000000000001 rpy=0 0 0
- joint radar_2: origin xyz=-0.3262 0.2262 0.217 rpy=0 0 0 -> xyz=-0.463200000000028 0.226199999999972 -0.0270000000000001 rpy=0 0 0
- joint radar_3: origin xyz=-0.13666 0 1.621 rpy=0 0 0 -> xyz=-0.27366 0 1.377 rpy=0 0 0
- joint wheel_1: limit (none) -> lower=0 upper=0 effort=0 velocity=0; origin xyz=0.29 0.1975 0.006 rpy=1.5708 0 3.1416 -> xyz=0 0 0.138999999999994 rpy=-1.5707963267949 0 0; parent base_link -> q_wheel_x_link; type continuous -> revolute
- joint wheel_2: axis 0 0 1 -> 0 0 -1; limit (none) -> lower=0 upper=0 effort=0 velocity=0; origin xyz=-0.29 -0.175 0.006 rpy=1.5708 -0.44445 3.1416 -> xyz=0 0 0.138999999999995 rpy=-1.5707963267949 0 0; parent base_link -> h_wheel_x_link; type continuous -> revolute
- joint wheel_3: origin xyz=0.29 0.1975 0.145 rpy=3.1416 0 3.1416 -> xyz=0.153 0.1975 -0.0990000000000054 rpy=3.14159265358979 0 3.14159265358979
- joint wheel_4: origin xyz=-0.29 -0.1975 0.145 rpy=3.1416 0 0 -> xyz=-0.427 -0.1975 -0.0990000000000054 rpy=3.14159265358979 0 0
- joint wheel_5: origin xyz=0.29 -0.1975 0.037 rpy=0 0 0 -> xyz=0.153 -0.1975 -0.207 rpy=0 0 0
- joint wheel_6: origin xyz=-0.29 0.1975 0.037 rpy=0 0 0 -> xyz=-0.427 0.1975 -0.207 rpy=0 0 0

File: jaka_kargo_ros2/src/jaka_kargo_moveit_config/config/jaka_kargo.ros2_control.xacro (robot description, xacro)
@@ -21,32 +21,4 @@
             </hardware>
             <!-- Joint interfaces generated for each joint -->
-            <joint name="body_j1">
-                <command_interface name="position"/>
-                <state_interface name="position">
-                  <param name="initial_value">${initial_positions['body_j1']}</param>
-                </state_interface>
-                <state_interface name="velocity"/>
-            </joint>
-            <joint name="body_j2">
-                <command_interface name="position"/>
-                <state_interface name="position">
-                  <param name="initial_value">${initial_positions['body_j2']}</param>
-                </state_interface>
-                <state_interface name="velocity"/>
-            </joint>
-            <joint name="body_j3">
-                <command_interface name="position"/>
-                <state_interface name="position">
-                  <param name="initial_value">${initial_positions['body_j3']}</param>
-                </state_interface>
-                <state_interface name="velocity"/>
-            </joint>
-            <joint name="body_j4">
-                <command_interface name="position"/>
-                <state_interface name="position">
-                  <param name="initial_value">${initial_positions['body_j4']}</param>
-                </state_interface>
-                <state_interface name="velocity"/>
-            </joint>
             <joint name="arm_lj1">
                 <command_interface name="position"/>
@@ -147,4 +119,53 @@
                 <state_interface name="velocity"/>
             </joint>
+            <joint name="body_j1">
+                <command_interface name="position"/>
+                <state_interface name="position">
+                  <param name="initial_value">${initial_positions['body_j1']}</param>
+                </state_interface>
+                <state_interface name="velocity"/>
+            </joint>
+            <joint name="body_j2">
+                <command_interface name="position"/>
+                <state_interface name="position">
+                  <param name="initial_value">${initial_positions['body_j2']}</param>
+                </state_interface>
+                <state_interface name="velocity"/>
+            </joint>
+            <joint name="body_j3">
+                <command_interface name="position"/>
+                <state_interface name="position">
+                  <param name="initial_value">${initial_positions['body_j3']}</param>
+                </state_interface>
+                <state_interface name="velocity"/>
+            </joint>
+            <joint name="body_j4">
+                <command_interface name="position"/>
+                <state_interface name="position">
+                  <param name="initial_value">${initial_positions['body_j4']}</param>
+                </state_interface>
+                <state_interface name="velocity"/>
+            </joint>
+            <joint name="agv_x">
+                <command_interface name="position"/>
+                <state_interface name="position">
+                  <param name="initial_value">${initial_positions['agv_x']}</param>
+                </state_interface>
+                <state_interface name="velocity"/>
+            </joint>
+            <joint name="agv_y">
+                <command_interface name="position"/>
+                <state_interface name="position">
+                  <param name="initial_value">${initial_positions['agv_y']}</param>
+                </state_interface>
+                <state_interface name="velocity"/>
+            </joint>
+            <joint name="agv_yaw">
+                <command_interface name="position"/>
+                <state_interface name="position">
+                  <param name="initial_value">${initial_positions['agv_yaw']}</param>
+                </state_interface>
+                <state_interface name="velocity"/>
+            </joint>
         </ros2_control>
     </xacro:macro>
